Commit message: legs

File: body.urdf (robot description, URDF)
Before this commit: robot robot, 3 links, 2 joints
Links:
- added link LeftLeg, mass 1; collision box size=1 0.25 0.25; visual box size=1 0.25 0.25
- added link LowerBackLeg, mass 1; collision box size=0.25 0.25 1; visual box size=0.25 0.25 1
- added link LowerFrontLeg, mass 1; collision box size=0.25 0.25 1; visual box size=0.25 0.25 1
- added link LowerLeftLeg, mass 1; collision box size=0.25 0.25 1; visual box size=0.25 0.25 1
- added link LowerRightLeg, mass 1; collision box size=0.25 0.25 1; visual box size=0.25 0.25 1
- added link RightLeg, mass 1; collision box size=1 0.25 0.25; visual box size=1 0.25 0.25
- link BackLeg: geometry collision box size=0.25 1 0.25; visual box size=0.25 1 0.25
- link FrontLeg: geometry collision box size=0.25 1 0.25; visual box size=0.25 1 0.25
Joints:
- added joint BackLeg_LowerBackLeg: type revolute, parent BackLeg, child LowerBackLeg, origin xyz=0 -1 0 rpy=0 0 0, axis 0 0 1, limit lower=-3.14159 upper=3.14159 effort=0.0 velocity=0.0
- added joint FrontLeg_LowerFrontLeg: type revolute, parent FrontLeg, child LowerFrontLeg, origin xyz=0 1 0 rpy=0 0 0, axis 0 0 1, limit lower=-3.14159 upper=3.14159 effort=0.0 velocity=0.0
- added joint LeftLeg_LowerLeftLeg: type revolute, parent LeftLeg, child LowerLeftLeg, origin xyz=-1 0 0 rpy=0 0 0, axis 0 0 1, limit lower=-3.14159 upper=3.14159 effort=0.0 velocity=0.0
- added joint RightLeg_LowerRightLeg: type revolute, parent RightLeg, child LowerRightLeg, origin xyz=1 0 0 rpy=0 0 0, axis 0 0 1, limit lower=-3.14159 upper=3.14159 effort=0.0 velocity=0.0
- added joint Torso_LeftLeg: type revolute, parent Torso, child LeftLeg, origin xyz=-0.5 0 1 rpy=0 0 0, axis 0 1 0, limit lower=-3.14159 upper=3.14159 effort=0.0 velocity=0.0
- added joint Torso_RightLeg: type revolute, parent Torso, child RightLeg, origin xyz=0.5 0 1 rpy=0 0 0, axis 0 1 0, limit lower=-3.14159 upper=3.14159 effort=0.0 velocity=0.0
- joint Torso_BackLeg: axis 0 1 0 -> 1 0 0; origin xyz=-0.5 0 1 rpy=0 0 0 -> xyz=0 -0.5 1 rpy=0 0 0
- joint Torso_FrontLeg: axis 0 1 0 -> 1 0 0; origin xyz=0.5 0 1 rpy=0 0 0 -> xyz=0 0.5 1 rpy=0 0 0

Commit message: evolving quad

File: body.urdf (robot description, URDF)
Before this commit: robot robot, 9 links, 8 joints
Joints:
- joint BackLeg_LowerBackLeg: axis 0 0 1 -> 1 0 0
- joint FrontLeg_LowerFrontLeg: axis 0 0 1 -> 1 0 0
- joint LeftLeg_LowerLeftLeg: axis 0 0 1 -> 0 1 0
- joint RightLeg_LowerRightLeg: axis 0 0 1 -> 0 1 0
